File: hardware/kicad/CARDio.kicad_pcb (KiCad board)
At the start: 4 copper layers, 85.6 x 54 mm, 53 parts, among them U1 ESP32-C3FH4, U2 MAX30102EFD+T_C6454833, U3 40MHz, U4 AMS1117-3.3_C347222, U5 AMS1117-1.8_C5250991

Commit message: Add KiCad schematic, project libraries and schematic/PCB sync
- kicad/CARDio.kicad_sch: imported from EasyEDA, then repaired by
  tools/fix_easyeda_schematic.py: 32 missing junctions (13 nets were
  split), real electrical pin types + PWR_FLAG, no-connect flags, power
  LED named PWR to match the PCB/BOM, page frame kept out of the BOM.
- Project-local libraries: CARDio.kicad_sym (deduplicated symbols) and
  CARDio.pretty (footprints, variants kept apart), with lib tables.
- tools/sync_pcb_from_schematic.py: board nets renamed to the
  schematic's and part fields copied onto footprints (no copper change).
- Results: ERC 0 errors, DRC 0 errors / 0 unconnected, schematic parity
  0 issues; Gerbers still match the production set.
- CARDio_schematic.pdf and updated hardware README.

Co-Authored-By: Claude Opus 5.5 <noreply@anthropic.com>
Parts:
- removed the PWR at (113.1, 87.6)
- added PWR: A-SP192DGHC-C01-4T, CARDio:LED0603-FD, F.Cu at (113.1, 87.6)
- ANT1: footprint WIFI ANTENNA MIFA INVERTED F ANTENNA -> CARDio:WIFI_ANTENNA_MIFA_INVERTED_F_ANTENNA
- C1, C12, C13, C14, C5, C6, C8: footprint C0603 -> CARDio:C0603
- C10, C11, C3, C4: footprint C0402 -> CARDio:C0402
- C15, C16, C18, C19, C20, C9: footprint C1206 -> CARDio:C1206
- C17, C2, C7: footprint C0805 -> CARDio:C0805
- D1: footprint SOT-23-6_L2.9-W1.6-P0.95-LS2.8-BL -> CARDio:SOT-23-6_L2.9-W1.6-P0.95-LS2.8-BL
- L1: footprint L0201 -> CARDio:L0201
- L3, L4: footprint L0402 -> CARDio:L0402
- LED1, LED10, LED12, LED2, LED3, LED4, LED5, LED6, LED7, LED8, LED9: footprint LED-SMD_4P-L2.0-W2.0-TL_WS2812B-2020 -> CARDio:LED-SMD_4P-L2.0-W2.0-TL_WS2812B-2020
- LED13, LED14: footprint LED-SMD_4P-L2.0-W2.0-TL_WS2812B-2020 -> CARDio:LED-SMD_4P-L2.0-W2.0-TL_WS2812B-2020_v2
- R1: footprint R0402 -> CARDio:R0402
- R2, R3, R4, R5, R6, R7, R8: footprint R0603 -> CARDio:R0603
- U1: footprint QFN-32_L5.0-W5.0-P0.50-TL-EP3.7 -> CARDio:QFN-32_L5.0-W5.0-P0.50-TL-EP3.7
- U2: footprint OESIP-14_L5.6-W3.3-P0.80-TL -> CARDio:OESIP-14_L5.6-W3.3-P0.80-TL
- U3: footprint CRYSTAL-SMD_4P-L3.2-W2.5-BL -> CARDio:CRYSTAL-SMD_4P-L3.2-W2.5-BL
- U4: footprint SOT-223-4_L6.5-W3.5-P2.30-LS7.0-BR -> CARDio:SOT-223-4_L6.5-W3.5-P2.30-LS7.0-BR
- U5: footprint SOT-223-3_L6.7-W3.7-P2.30-LS7.0-BR -> CARDio:SOT-223-3_L6.7-W3.7-P2.30-LS7.0-BR
- USB1: footprint USB-C-SMD_TYPE-C-6PIN-2MD-073 -> CARDio:USB-C-SMD_TYPE-C-6PIN-2MD-073
Connections:
- net ANT1_ANT renamed Net-(ANT1-PadANT)
- net LED12_1 renamed Net-(LED12-DO)
- net LED13_1 renamed Net-(LED13-DO)
- net LED1_1 renamed Net-(LED1-DO)
- net LED2_1 renamed Net-(LED2-DO)
- net LED3_1 renamed Net-(LED1-DI)
- net LED3_3 renamed Net-(LED10-DO)
- net LED4_1 renamed Net-(LED4-DO)
- net LED5_1 renamed Net-(LED5-DO)
- net LED5_3 renamed Net-(LED5-DI)
- net LED7_1 renamed Net-(LED7-DO)
- net LED8_1 renamed Net-(LED12-DI)
- net LED9_1 renamed Net-(LED10-DI)
- net U1_1 renamed Net-(U1-LNA_IN)
- net U1_2 renamed Net-(C7-Pad2)
- net U1_28 renamed Net-(U1-U0TXD)
- net U1_29 renamed Net-(U1-XTAL_N)
- net U1_30 renamed Net-(U1-XTAL_P)
- net U1_7 renamed Net-(U1-CHIP_EN)
- net U2_13 renamed Net-(U2-INT#)
- net U3_1 renamed Net-(C3-Pad1)
- net USB1_10 renamed Net-(USB1-CC2)
- net USB1_4 renamed Net-(USB1-CC1)
- net USB1_5 renamed Net-(USB1-DN1)
- net USB1_6 renamed Net-(USB1-DP1)
- LED14 pad 1: LED14_1 -> unconnected-(LED14-DO-Pad1)
- R8 pad 2: LED11_1 -> Net-(PWR-A)
- U1 pad 18: U1_18 -> unconnected-(U1-VDD_SPI-Pad18)
- U1 pad 19: U1_19 -> unconnected-(U1-SPIHD-Pad19)
- U1 pad 20: U1_20 -> unconnected-(U1-SPIWP-Pad20)
- U1 pad 21: U1_21 -> unconnected-(U1-SPICS0-Pad21)
- U1 pad 22: U1_22 -> unconnected-(U1-SPICLK-Pad22)
- U1 pad 23: U1_23 -> unconnected-(U1-SPID-Pad23)
- U1 pad 24: U1_24 -> unconnected-(U1-SPIQ-Pad24)
- U2 pad 1: U2_1 -> unconnected-(U2-N.C.-Pad1)
- U2 pad 14: U2_14 -> unconnected-(U2-N.C.-Pad14)
- U2 pad 5: U2_5 -> unconnected-(U2-N.C.-Pad5)
- U2 pad 6: U2_6 -> unconnected-(U2-N.C.-Pad6)
- U2 pad 7: U2_7 -> unconnected-(U2-N.C.-Pad7)
- U2 pad 8: U2_8 -> unconnected-(U2-N.C.-Pad8)
- U4 pad 4: U4_4 -> unconnected-(U4-TAB-Pad4)
- USB1 pad 13: USB1_13 -> unconnected-(USB1-SHELL-Pad13)
- USB1 pad 14: USB1_14 -> unconnected-(USB1-SHELL-Pad14)
- USB1 pad 3: USB1_3 -> unconnected-(USB1-SBU2-Pad3)
- USB1 pad 9: USB1_9 -> unconnected-(USB1-SBU1-Pad9)
Routing:
- net unconnected-(USB1-SHELL-Pad14): track 0.00 -> 4.20 mm
- net unconnected-(USB1-SHELL-Pad13): track 0.00 -> 4.20 mm
- net USB1_14: track 4.20 -> 0.00 mm
- net USB1_13: track 4.20 -> 0.00 mm
- net Net-(PWR-A): track 0.00 -> 3.22 mm
- net LED11_1: track 3.22 -> 0.00 mm
